Commit message: nav2 syntax update for plugins in Jazzy

File: config/robot_description/pioneer2dx/body.xacro (robot description, xacro)
@@ -170,5 +170,5 @@
   <link name="base_laser"/>
   <joint name="top_to_laser_joint" type="fixed">
-    <origin xyz="0 0 ${laser_z}" rpy="0 0 0"/>
+    <origin xyz="0 0 ${laser_z}" rpy="0 0 ${M_PI}"/>
     <parent link="top_plate"/>
     <child  link="base_laser"/>

Commit message: pkg renamed

File: config/robot_description/pioneer2dx/body.xacro (robot description, xacro)
@@ -1,5 +1,5 @@
 <?xml version="1.0"?>
 <robot xmlns:xacro="http://ros.org/wiki/xacro">
-  <xacro:include filename="$(find tuw2_launches)/config/robot_description/pioneer2dx/wheel.xacro"/>
+  <xacro:include filename="$(find tuw_bringup)/config/robot_description/pioneer2dx/wheel.xacro"/>
   <material name="ChassisRed"  ><color rgba="0.851 0.0 0.0 1.0"/></material>
   <material name="TopBlack"    ><color rgba="0.038 0.038 0.038 1.0"/></material>
@@ -19,5 +19,5 @@
       <origin xyz="-0.045 0 0.148" rpy="0 0 0"/>
       <geometry>
-        <mesh filename="package://tuw2_launches/config/robot_description/pioneer2dx/meshes/chassis.stl"/>
+        <mesh filename="package://tuw_bringup/config/robot_description/pioneer2dx/meshes/chassis.stl"/>
       </geometry>
       <material name="ChassisRed"/>
@@ -45,5 +45,5 @@
       <origin xyz="0 0 0" rpy="0 0 0"/>
       <geometry>
-        <mesh filename="package://tuw2_launches/config/robot_description/pioneer2dx/meshes/top.stl"/>
+        <mesh filename="package://tuw_bringup/config/robot_description/pioneer2dx/meshes/top.stl"/>
       </geometry>
       <material name="TopBlack"/>
@@ -64,5 +64,5 @@
       <origin xyz="0 0 0" rpy="0 0 0"/>
       <geometry>
-        <mesh filename="package://tuw2_launches/config/robot_description/pioneer2dx/meshes/swivel.stl"/>
+        <mesh filename="package://tuw_bringup/config/robot_description/pioneer2dx/meshes/swivel.stl"/>
       </geometry>
       <material name="Swivel"/>
@@ -88,5 +88,5 @@
       <origin xyz="0 0 0" rpy="0 0 0"/>
       <geometry>
-        <mesh filename="package://tuw2_launches/config/robot_description/pioneer2dx/meshes/center_wheel.stl"/>
+        <mesh filename="package://tuw_bringup/config/robot_description/pioneer2dx/meshes/center_wheel.stl"/>
       </geometry>
       <material name="WheelBlack"/>
@@ -118,5 +118,5 @@
       <origin xyz="0 0 0" rpy="0 0 0"/>
       <geometry>
-        <mesh filename="package://tuw2_launches/config/robot_description/pioneer2dx/meshes/center_hubcap.stl"/>
+        <mesh filename="package://tuw_bringup/config/robot_description/pioneer2dx/meshes/center_hubcap.stl"/>
       </geometry>
       <material name="Swivel"/>
@@ -139,5 +139,5 @@
       <origin xyz="0 0 0" rpy="0 0 0"/>
       <geometry>
-        <mesh filename="package://tuw2_launches/config/robot_description/pioneer2dx/meshes/front_sonar.stl"/>
+        <mesh filename="package://tuw_bringup/config/robot_description/pioneer2dx/meshes/front_sonar.stl"/>
       </geometry>
       <material name="SonarYellow"/>
@@ -158,5 +158,5 @@
       <origin xyz="0 0 0" rpy="0 0 0"/>
       <geometry>
-        <mesh filename="package://tuw2_launches/config/robot_description/pioneer2dx/meshes/back_sonar.stl"/>
+        <mesh filename="package://tuw_bringup/config/robot_description/pioneer2dx/meshes/back_sonar.stl"/>
       </geometry>
       <material name="SonarYellow"/>

File: config/robot_description/pioneer2dx/main.xacro (robot description, xacro)
@@ -3,4 +3,4 @@
   <xacro:property name="M_PI" value="3.14159265358979"/>
   <xacro:property name="laser_z" value="0.07"/>
-  <xacro:include filename="$(find tuw2_launches)/config/robot_description/pioneer2dx/body.xacro"/>
+  <xacro:include filename="$(find tuw_bringup)/config/robot_description/pioneer2dx/body.xacro"/>
 </robot>

File: config/robot_description/pioneer2dx/wheel.xacro (robot description, xacro)
@@ -13,5 +13,5 @@
         <origin xyz="0 0 0" rpy="0 0 0"/>
         <geometry>
-          <mesh filename="package://tuw2_launches/config/robot_description/pioneer2dx/meshes/${suffix}_wheel.stl"/>
+          <mesh filename="package://tuw_bringup/config/robot_description/pioneer2dx/meshes/${suffix}_wheel.stl"/>
         </geometry>
         <material name="WheelBlack"/>
@@ -35,5 +35,5 @@
         <origin xyz="0 0 0" rpy="0 0 0"/>
         <geometry>
-          <mesh filename="package://tuw2_launches/config/robot_description/pioneer2dx/meshes/${suffix}_hubcap.stl"/>
+          <mesh filename="package://tuw_bringup/config/robot_description/pioneer2dx/meshes/${suffix}_hubcap.stl"/>
         </geometry>
         <material name="HubcapYellow"/>

Commit message: base_laser renamed to laser0 and scan to scan_raw with laser_filter activ

File: config/robot_description/pioneer2dx/body.xacro (robot description, xacro)
@@ -168,9 +168,9 @@
     <child  link="back_sonar"/>
   </joint>
-  <link name="base_laser"/>
+  <link name="laser0"/>
   <joint name="top_to_laser_joint" type="fixed">
     <origin xyz="0 0 ${laser_z}" rpy="0 0 ${M_PI}"/>
     <parent link="top_plate"/>
-    <child  link="base_laser"/>
+    <child  link="laser0"/>
   </joint>
 </robot>
